File: board_fille/ivegotdapower-elec.kicad_pcb (KiCad board)
At the start: 2 copper layers, 44.5 x 20.3 mm, 16 parts, among them J1 Conn_02x03_Odd_Even, J2 Conn_02x03_Odd_Even, U1 LM2596S-ADJ

Commit message: Silkscreen, better pcb
Parts:
- moved R6 3.13 mm to (110.7, 115.7), turned to 0 degrees
- moved C3 0.07 mm to (124.4, 103.6)
Routing:
- net /on-off: track 14.1 -> 15.0 mm
Other:
- outline, holes or cut-outs redrawn
- board text added: "In"
- board text added: "Out"
- board text added: "Status"
